Commit message: imported modified stand_chest into project

File: Assets/URDF/gopher_old.xacro (robot description, xacro)
@@ -15,15 +15,12 @@
     <!-- Include files -->
     <xacro:include filename="$(find gopher_description)/fetch_description/urdf/freight.urdf.xacro" />
-    <!-- <xacro:include filename="$(find gopher_description)/torso_description/urdf/torso.urdf.xacro" /> -->
+    <xacro:include filename="$(find gopher_description)/torso_description/urdf/torso.urdf.xacro" />
     <xacro:include filename="$(find gopher_description)/realsense2_description/urdf/_d435.urdf.xacro" />
     <xacro:include filename="$(find gopher_description)/kortex_description/arms/urdf/kortex_robot.xacro" />
-    <xacro:include filename="$(find gopher_description)/stand_chest_description/urdf/stand_chest.xacro" />
     <!-- Load urdf -->
     <!-- base -->
     <xacro:load_freight_urdf prefix="$(arg prefix)" />
     <!-- torso -->
-    <!-- <xacro:load_torso_urdf prefix="$(arg prefix)" parent="$(arg prefix)chassis_link" /> -->
-    <!-- stand_chest -->
-    <xacro:load_stand_chest_urdf prefix="$(arg prefix)" parent="$(arg prefix)chassis_link" />
+    <xacro:load_torso_urdf prefix="$(arg prefix)" parent="$(arg prefix)chassis_link" />
     <!-- main camera -->
     <xacro:sensor_d435 prefix="$(arg prefix)main_cam_" parent="$(arg prefix)main_cam_pitch_link">
@@ -34,11 +31,11 @@
         <xacro:load_kortex arm="$(arg arm)" gripper="$(arg gripper)" dof="$(arg dof)"
                            vision="$(arg vision)" sim="$(arg sim)"
-                           prefix="$(arg right_prefix)" parent="$(arg prefix)right_mounting_plate">
-            <origin xyz="0.05 -0.075 0.01" rpy="0 0 0" />
+                           prefix="$(arg right_prefix)" parent="$(arg prefix)torso">
+            <origin xyz="-0.03 -0.03 0.7" rpy="1.5708 0 0" />
         </xacro:load_kortex>
         <xacro:load_kortex arm="$(arg arm)" gripper="$(arg gripper)" dof="$(arg dof)"
                            vision="$(arg vision)" sim="$(arg sim)"
-                           prefix="$(arg left_prefix)" parent="$(arg prefix)left_mounting_plate">
-            <origin xyz="0.05 0.075 0.01" rpy="0 0 3.1416" />
+                           prefix="$(arg left_prefix)" parent="$(arg prefix)torso">
+            <origin xyz="-0.03 0.03 0.7" rpy="1.5708 0 3.1416" />
         </xacro:load_kortex>
     </xacro:if>
@@ -48,8 +45,6 @@
         <xacro:include filename="$(find gopher_description)/torso_description/urdf/torso.gazebo.xacro" />
         <xacro:include filename="$(find gopher_description)/realsense2_description/urdf/_d435.gazebo.xacro" />
-        <xacro:include filename="$(find gopher_description)/stand_chest_description/urdf/stand_chest.gazebo.xacro" />
         <xacro:load_freight_gazebo prefix="$(arg prefix)" />
-        <!-- <xacro:load_torso_gazebo prefix="$(arg prefix)" /> -->
-        <xacro:load_stand_chest_gazebo prefix="$(arg prefix)" />
+        <xacro:load_torso_gazebo prefix="$(arg prefix)" />
         <xacro:gazebo_d435 camera_name="main_cam" reference_link="$(arg prefix)main_cam_link"
                            frame_name="main_cam_color_optical_frame"
