Commit message: added chest to hello prefab

File: Assets/URDF/gopher.urdf (robot description, URDF)
Before this commit: robot Gopher, 64 links, 63 joints
Links:
- removed link gopher/torso
- added link gopher/chest, mass 16.262774451109365; collision mesh filename=package://gopher_description/stand_chest_description/meshes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; visual mesh filename=package://gopher_description/stand_chest_description/meshes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
- added link gopher/left_mounting_plate, mass 0.39829293027064805; collision mesh filename=package://gopher_description/stand_chest_description/meshes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; visual mesh filename=package://gopher_description/stand_chest_description/meshes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
- added link gopher/right_mounting_plate, mass 0.39829293027064405; collision mesh filename=package://gopher_description/stand_chest_description/meshes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; visual mesh filename=package://gopher_description/stand_chest_description/meshes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
- added link gopher/stand, mass 33.86884985630993; collision mesh filename=package://gopher_description/stand_chest_description/meshes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; visual mesh filename=package://gopher_description/stand_chest_description/meshes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
- link gopher/left_arm_camera_color_frame: mass 0.001 -> None
- link gopher/left_arm_camera_depth_frame: mass 0.001 -> None
- link gopher/left_arm_camera_link: mass 0.001 -> None
- link gopher/left_arm_end_effector_link: mass 0.001 -> None
- link gopher/left_arm_left_inner_finger_pad: mass 0.001 -> None
- link gopher/left_arm_right_inner_finger_pad: mass 0.001 -> None
- link gopher/left_arm_tool_frame: mass 0.001 -> None
- link gopher/right_arm_camera_color_frame: mass 0.001 -> None
- link gopher/right_arm_camera_depth_frame: mass 0.001 -> None
- link gopher/right_arm_camera_link: mass 0.001 -> None
- link gopher/right_arm_end_effector_link: mass 0.001 -> None
- link gopher/right_arm_left_inner_finger_pad: mass 0.001 -> None
- link gopher/right_arm_right_inner_finger_pad: mass 0.001 -> None
- link gopher/right_arm_tool_frame: mass 0.001 -> None
Joints:
- removed joint gopher/torso_joint
- added joint gopher/chest_joint: type prismatic, parent gopher/stand, child gopher/chest, origin xyz=-0.082038 0.000502 0.303534 rpy=0 0 0, axis 0.0 0.0 1.0, limit lower=0.00 upper=0.47 effort=1000000 velocity=0.5
- added joint gopher/stand_joint: type fixed, parent gopher/chassis_link, child gopher/stand, origin xyz=-0.1 0.0 0.357425 rpy=0 0 0
- added joint left_mounting_plate_joint: type fixed, parent gopher/chest, child gopher/left_mounting_plate, origin xyz=0.162 0.08192 0.267206 rpy=0 0 0
- added joint right_mounting_plate_joint: type fixed, parent gopher/chest, child gopher/right_mounting_plate, origin xyz=0.162 -0.08192 0.267206 rpy=0 0 0
- joint gopher/left_arm_finger_joint: origin xyz=0 -0.0306011 0.054904 rpy=0 0 3.14159265359 -> xyz=0 -0.0306011 0.054904 rpy=0 0 3.141592653589793
- joint gopher/left_arm_left_inner_knuckle_joint: origin xyz=0 -0.0127 0.06142 rpy=0 0 3.14159265359 -> xyz=0 -0.0127 0.06142 rpy=0 0 3.141592653589793
- joint gopher/left_arm_shoulder_to_arm_root: origin xyz=-0.03 0.03 0.7 rpy=1.5708 0 3.1416 -> xyz=0.00 0.06 -0.04 rpy=0 0.78539 1.5707; parent gopher/torso -> gopher/left_mounting_plate
- joint gopher/main_cam_support_joint: origin xyz=0.0 0.0 0.8 rpy=0 0 0 -> xyz=0.16 0.0 0.46 rpy=0 0 0; parent gopher/torso -> gopher/chest
- joint gopher/right_arm_finger_joint: origin xyz=0 -0.0306011 0.054904 rpy=0 0 3.14159265359 -> xyz=0 -0.0306011 0.054904 rpy=0 0 3.141592653589793
- joint gopher/right_arm_left_inner_knuckle_joint: origin xyz=0 -0.0127 0.06142 rpy=0 0 3.14159265359 -> xyz=0 -0.0127 0.06142 rpy=0 0 3.141592653589793
- joint gopher/right_arm_shoulder_to_arm_root: origin xyz=-0.03 -0.03 0.7 rpy=1.5708 0 0 -> xyz=0 -0.06 -0.04 rpy=0 0.78539 -1.5707; parent gopher/torso -> gopher/right_mounting_plate

File: Assets/URDF/gopher.xacro (robot description, xacro)
@@ -35,10 +35,10 @@
                            vision="$(arg vision)" sim="$(arg sim)"
                            prefix="$(arg right_prefix)" parent="$(arg prefix)right_mounting_plate">
-            <origin xyz="0.05 -0.075 0.01" rpy="0 0 0" />
+            <origin xyz="0 -0.06 -0.04" rpy="0 0.78539 -1.5707" />
         </xacro:load_kortex>
         <xacro:load_kortex arm="$(arg arm)" gripper="$(arg gripper)" dof="$(arg dof)"
                            vision="$(arg vision)" sim="$(arg sim)"
                            prefix="$(arg left_prefix)" parent="$(arg prefix)left_mounting_plate">
-            <origin xyz="0.05 0.075 0.01" rpy="0 0 3.1416" />
+            <origin xyz="0.00 0.06 -0.04" rpy="0 0.78539 1.5707" />
         </xacro:load_kortex>
     </xacro:if>

File: Assets/URDF/gopher_description/stand_chest_description/urdf/stand_chest.xacro (robot description, xacro)
@@ -190,5 +190,5 @@
       <parent link="${prefix}chest"/>
       <child link="${prefix}main_cam_support"/>
-      <origin rpy="0 0 0" xyz="0.0 0.0 0.8"/>
+      <origin rpy="0 0 0" xyz="0.16 0.0 0.46"/>
       <axis xyz="0 0 1"/>
     </joint>
