Commit message: update robot with motorized chest

File: Assets/URDF/gopher_old.urdf (robot description, URDF)
Before this commit: robot Gopher, 67 links, 66 joints
Links:
- removed link gopher/chest
- removed link gopher/left_mounting_plate
- removed link gopher/right_mounting_plate
- removed link gopher/stand
- added link gopher/torso, mass 12.0; collision mesh filename=package://gopher_description/torso_description/meshes/torso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; visual mesh filename=package://gopher_description/torso_description/meshes/torso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
- link gopher/left_arm_camera_color_frame: mass None -> 0.001
- link gopher/left_arm_camera_depth_frame: mass None -> 0.001
- link gopher/left_arm_camera_link: mass None -> 0.001
- link gopher/left_arm_end_effector_link: mass None -> 0.001
- link gopher/left_arm_left_inner_finger_pad: mass None -> 0.001
- link gopher/left_arm_right_inner_finger_pad: mass None -> 0.001
- link gopher/left_arm_tool_frame: mass None -> 0.001
- link gopher/right_arm_camera_color_frame: mass None -> 0.001
- link gopher/right_arm_camera_depth_frame: mass None -> 0.001
- link gopher/right_arm_camera_link: mass None -> 0.001
- link gopher/right_arm_end_effector_link: mass None -> 0.001
- link gopher/right_arm_left_inner_finger_pad: mass None -> 0.001
- link gopher/right_arm_right_inner_finger_pad: mass None -> 0.001
- link gopher/right_arm_tool_frame: mass None -> 0.001
Joints:
- removed joint gopher/chest_joint
- removed joint gopher/stand_joint
- removed joint left_mounting_plate_joint
- removed joint right_mounting_plate_joint
- added joint gopher/torso_joint: type fixed, parent gopher/chassis_link, child gopher/torso, origin xyz=-0.0 0 0.36 rpy=0 0 0, axis 0 0 1
- joint gopher/left_arm_finger_joint: origin xyz=0 -0.0306011 0.054904 rpy=0 0 3.141592653589793 -> xyz=0 -0.0306011 0.054904 rpy=0 0 3.14159265359
- joint gopher/left_arm_left_inner_knuckle_joint: origin xyz=0 -0.0127 0.06142 rpy=0 0 3.141592653589793 -> xyz=0 -0.0127 0.06142 rpy=0 0 3.14159265359
- joint gopher/left_arm_shoulder_to_arm_root: origin xyz=0.00 0.06 -0.04 rpy=0 0.78539 1.5707 -> xyz=-0.03 0.03 0.7 rpy=1.5708 0 3.1416; parent gopher/left_mounting_plate -> gopher/torso
- joint gopher/main_cam_support_joint: origin xyz=0.16 0.0 0.46 rpy=0 0 0 -> xyz=0.0 0.0 0.8 rpy=0 0 0; parent gopher/chest -> gopher/torso
- joint gopher/right_arm_finger_joint: origin xyz=0 -0.0306011 0.054904 rpy=0 0 3.141592653589793 -> xyz=0 -0.0306011 0.054904 rpy=0 0 3.14159265359
- joint gopher/right_arm_left_inner_knuckle_joint: origin xyz=0 -0.0127 0.06142 rpy=0 0 3.141592653589793 -> xyz=0 -0.0127 0.06142 rpy=0 0 3.14159265359
- joint gopher/right_arm_shoulder_to_arm_root: origin xyz=0 -0.06 -0.04 rpy=0 0.78539 -1.5707 -> xyz=-0.03 -0.03 0.7 rpy=1.5708 0 0; parent gopher/right_mounting_plate -> gopher/torso
